File: kicad/blinkencard_frontpanel.sch (KiCad schematic (older format))
At the start: 62 parts, among them Q1 BC847, Q2 BC847, Q3 BC847, Q4 BC847, Q5 BC847, SW1 LEFT, SW2 1, SW3 0, SW4 RIGHT

Commit message: Use CP2102A USB-UART and GPIO instead of ESP32 to keep it simple. Add power section and start routing.
Parts:
- D10, D11, D12, D13, D14, D15, D16, D17, D20, D21, D22, D23, D24, D25, D26, D27, D30, D31, D32, D33, D34, D35, D36, D37, D40, D41, D42, D43, D44, D45, D46, D47, D50, D51, D52, D53, D54, D55, D56, D57: footprint LED_SMD:LED_0805_2012Metric -> LED_SMD:LED_1206_3216Metric_ReverseMount_Hole1.8x2.4mm
- SW1: renamed from SW3; footprint Button_Switch_THT:SW_PUSH_6mm_H5mm -> Button_Switch_SMD:SW_SPST_PTS645
- SW2, SW4: footprint Button_Switch_THT:SW_PUSH_6mm_H5mm -> Button_Switch_SMD:SW_SPST_PTS645
- SW3: renamed from SW1; footprint Button_Switch_THT:SW_PUSH_6mm_H5mm -> Button_Switch_SMD:SW_SPST_PTS645
Other:
- moved on the sheet: SW1, SW2

Commit message: Update blinkencard_frontpanel.sch
Parts:
- D10, D11, D12, D13, D14, D15, D16, D17, D20, D21, D22, D23, D24, D25, D26, D27, D30, D31, D32, D33, D34, D35, D36, D37, D40, D41, D42, D43, D44, D45, D46, D47, D50, D51, D52, D53, D54, D55, D56, D57: footprint LED_SMD:LED_1206_3216Metric_ReverseMount_Hole1.8x2.4mm -> blinkencard:LED_1206_3216Metric_ReverseMount_Hole1.8x2.4mm

Commit message: Move buttons to more sensible locations, finalize silk, tape out v1.0
Parts:
- R1, R2, R3, R4, R5: value 1k -> 10k
- R10, R11, R12, R13, R14, R15, R16, R17: value 330 -> 270
Changed lines of the file:
@@
 P 2700 4300
 F 0 "R17" H 2768 4300 50  0000 L CNN
-F 1 "330" H 2768 4255 50  0001 L CNN
+F 1 "270" H 2768 4255 50  0001 L CNN
 F 2 "Resistor_SMD:R_0603_1608Metric" V 2740 4290 50  0001 C CNN
 F 3 "~" H 2700 4300 50  0001 C CNN
@@
 P 2950 4300
 F 0 "R16" H 3018 4300 50  0000 L CNN
-F 1 "330" H 3018 4255 50  0001 L CNN
+F 1 "270" H 3018 4255 50  0001 L CNN
 F 2 "Resistor_SMD:R_0603_1608Metric" V 2990 4290 50  0001 C CNN
 F 3 "~" H 2950 4300 50  0001 C CNN
@@
 P 3200 4300
 F 0 "R15" H 3268 4300 50  0000 L CNN
-F 1 "330" H 3268 4255 50  0001 L CNN
+F 1 "270" H 3268 4255 50  0001 L CNN
 F 2 "Resistor_SMD:R_0603_1608Metric" V 3240 4290 50  0001 C CNN
 F 3 "~" H 3200 4300 50  0001 C CNN
@@
 P 3450 4300
 F 0 "R14" H 3518 4300 50  0000 L CNN
-F 1 "330" H 3518 4255 50  0001 L CNN
+F 1 "270" H 3518 4255 50  0001 L CNN
 F 2 "Resistor_SMD:R_0603_1608Metric" V 3490 4290 50  0001 C CNN
 F 3 "~" H 3450 4300 50  0001 C CNN
@@
 P 3700 4300
 F 0 "R13" H 3768 4300 50  0000 L CNN
-F 1 "330" H 3768 4255 50  0001 L CNN
+F 1 "270" H 3768 4255 50  0001 L CNN
 F 2 "Resistor_SMD:R_0603_1608Metric" V 3740 4290 50  0001 C CNN
 F 3 "~" H 3700 4300 50  0001 C CNN
@@
 P 3950 4300
 F 0 "R12" H 4018 4300 50  0000 L CNN
-F 1 "330" H 4018 4255 50  0001 L CNN
+F 1 "270" H 4018 4255 50  0001 L CNN
 F 2 "Resistor_SMD:R_0603_1608Metric" V 3990 4290 50  0001 C CNN
 F 3 "~" H 3950 4300 50  0001 C CNN
@@
 P 4200 4300
 F 0 "R11" H 4268 4300 50  0000 L CNN
-F 1 "330" H 4268 4255 50  0001 L CNN
+F 1 "270" H 4268 4255 50  0001 L CNN
 F 2 "Resistor_SMD:R_0603_1608Metric" V 4240 4290 50  0001 C CNN
 F 3 "~" H 4200 4300 50  0001 C CNN
@@
 P 4450 4300
 F 0 "R10" H 4518 4300 50  0000 L CNN
-F 1 "330" H 4518 4255 50  0001 L CNN
+F 1 "270" H 4518 4255 50  0001 L CNN
 F 2 "Resistor_SMD:R_0603_1608Metric" V 4490 4290 50  0001 C CNN
 F 3 "~" H 4450 4300 50  0001 C CNN
@@
 P 1650 1500
 F 0 "R1" V 1537 1500 50  0000 C CNN
-F 1 "1k" V 1536 1500 50  0001 C CNN
+F 1 "10k" V 1536 1500 50  0001 C CNN
 F 2 "Resistor_SMD:R_0603_1608Metric" V 1690 1490 50  0001 C CNN
 F 3 "~" H 1650 1500 50  0001 C CNN
@@
 P 1650 2000
 F 0 "R2" V 1537 2000 50  0000 C CNN
-F 1 "1k" V 1536 2000 50  0001 C CNN
+F 1 "10k" V 1536 2000 50  0001 C CNN
 F 2 "Resistor_SMD:R_0603_1608Metric" V 1690 1990 50  0001 C CNN
 F 3 "~" H 1650 2000 50  0001 C CNN
@@
 P 1650 2500
 F 0 "R3" V 1537 2500 50  0000 C CNN
-F 1 "1k" V 1536 2500 50  0001 C CNN
+F 1 "10k" V 1536 2500 50  0001 C CNN
 F 2 "Resistor_SMD:R_0603_1608Metric" V 1690 2490 50  0001 C CNN
 F 3 "~" H 1650 2500 50  0001 C CNN
@@
 P 1650 3000
 F 0 "R4" V 1537 3000 50  0000 C CNN
-F 1 "1k" V 1536 3000 50  0001 C CNN
+F 1 "10k" V 1536 3000 50  0001 C CNN
 F 2 "Resistor_SMD:R_0603_1608Metric" V 1690 2990 50  0001 C CNN
 F 3 "~" H 1650 3000 50  0001 C CNN
@@
 P 1650 3500
 F 0 "R5" V 1537 3500 50  0000 C CNN
-F 1 "1k" V 1536 3500 50  0001 C CNN
+F 1 "10k" V 1536 3500 50  0001 C CNN
 F 2 "Resistor_SMD:R_0603_1608Metric" V 1690 3490 50  0001 C CNN
 F 3 "~" H 1650 3500 50  0001 C CNN

Commit message: Start v2.0 - change USB-UART to ESP32 and bugfixes
Parts:
- R1, R2, R3, R4, R5: value 10k -> 10K
Changed lines of the file:
@@
 P 1650 1500
 F 0 "R1" V 1537 1500 50  0000 C CNN
-F 1 "10k" V 1536 1500 50  0001 C CNN
+F 1 "10K" V 1536 1500 50  0001 C CNN
 F 2 "Resistor_SMD:R_0603_1608Metric" V 1690 1490 50  0001 C CNN
 F 3 "~" H 1650 1500 50  0001 C CNN
@@
 P 1650 2000
 F 0 "R2" V 1537 2000 50  0000 C CNN
-F 1 "10k" V 1536 2000 50  0001 C CNN
+F 1 "10K" V 1536 2000 50  0001 C CNN
 F 2 "Resistor_SMD:R_0603_1608Metric" V 1690 1990 50  0001 C CNN
 F 3 "~" H 1650 2000 50  0001 C CNN
@@
 P 1650 2500
 F 0 "R3" V 1537 2500 50  0000 C CNN
-F 1 "10k" V 1536 2500 50  0001 C CNN
+F 1 "10K" V 1536 2500 50  0001 C CNN
 F 2 "Resistor_SMD:R_0603_1608Metric" V 1690 2490 50  0001 C CNN
 F 3 "~" H 1650 2500 50  0001 C CNN
@@
 P 1650 3000
 F 0 "R4" V 1537 3000 50  0000 C CNN
-F 1 "10k" V 1536 3000 50  0001 C CNN
+F 1 "10K" V 1536 3000 50  0001 C CNN
 F 2 "Resistor_SMD:R_0603_1608Metric" V 1690 2990 50  0001 C CNN
 F 3 "~" H 1650 3000 50  0001 C CNN
@@
 P 1650 3500
 F 0 "R5" V 1537 3500 50  0000 C CNN
-F 1 "10k" V 1536 3500 50  0001 C CNN
+F 1 "10K" V 1536 3500 50  0001 C CNN
 F 2 "Resistor_SMD:R_0603_1608Metric" V 1690 3490 50  0001 C CNN
 F 3 "~" H 1650 3500 50  0001 C CNN

Commit message: v2.0 release - clean silk, add order number placeholder for JLCPCB, add MFG PN in components for BOM, add BOM, add STEP, generate fab outputs
Parts:
- D10, D11, D12, D13, D14, D15, D16, D17, D20, D21, D22, D23, D24, D25, D26, D27, D30, D31, D32, D33, D34, D35, D36, D37, D40, D41, D42, D43, D44, D45, D46, D47, D50, D51, D52, D53, D54, D55, D56, D57:  mfg_part (none) -> LTST-C230KRKT
- Q1, Q2, Q3, Q4, Q5:  mfg_part (none) -> BC847CLT1G
- R1, R2, R3, R4, R5:  mfg_part (none) -> RC0603JR-0710KL
- R10, R11, R12, R13, R14, R15, R16, R17:  mfg_part (none) -> RMCF0603JT270R
- SW1, SW2, SW3, SW4:  mfg_part (none) -> PTS645SM50SMTR92 LFS
